Commit message: Replace lidar scan localization with single depth camera scan localization

File: nav2_bringup/urdf/single_drum_roller.urdf (robot description, URDF)
Before this commit: robot turtlebot3_waffle, 13 links, 12 joints
Links:
- removed link base_scan
- added link camera_scan_frame
Joints:
- removed joint scan_joint
- added joint camera_scan_joint: type fixed, parent camera_link, child camera_scan_frame, origin xyz=0.005 0.028 0.013 rpy=0 0 0

Commit message: Rename camera to front_camera

File: nav2_bringup/urdf/single_drum_roller.urdf (robot description, URDF)
Before this commit: robot turtlebot3_waffle, 13 links, 12 joints
Links:
- removed link camera_depth_frame
- removed link camera_depth_optical_frame
- removed link camera_link
- removed link camera_rgb_frame
- removed link camera_rgb_optical_frame
- removed link camera_scan_frame
- added link front_camera_depth_frame
- added link front_camera_depth_optical_frame
- added link front_camera_link; collision box size=0.012 0.132 0.020; visual mesh filename=package://turtlebot3_gazebo/models/turtlebot3_common/meshes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
- added link front_camera_rgb_frame
- added link front_camera_rgb_optical_frame
- added link front_camera_scan_frame
Joints:
- removed joint camera_depth_joint
- removed joint camera_depth_optical_joint
- removed joint camera_joint
- removed joint camera_rgb_joint
- removed joint camera_rgb_optical_joint
- removed joint camera_scan_joint
- added joint front_camera_depth_joint: type fixed, parent front_camera_link, child front_camera_depth_frame, origin xyz=0.005 0.028 0.013 rpy=-1.57 0 -1.57
- added joint front_camera_depth_optical_joint: type fixed, parent front_camera_depth_frame, child front_camera_depth_optical_frame, origin xyz=0 0 0 rpy=0 0 0
- added joint front_camera_joint: type fixed, parent base_link, child front_camera_link, origin xyz=0.064 0 0.094 rpy=0 0 0
- added joint front_camera_rgb_joint: type fixed, parent front_camera_link, child front_camera_rgb_frame, origin xyz=0.005 0.018 0.013 rpy=0 0 0
- added joint front_camera_rgb_optical_joint: type fixed, parent front_camera_rgb_frame, child front_camera_rgb_optical_frame, origin xyz=0 0 0 rpy=-1.57 0 -1.57
- added joint front_camera_scan_joint: type fixed, parent front_camera_link, child front_camera_scan_frame, origin xyz=0.005 0.028 0.013 rpy=0 0 0

Commit message: Add rear camera for perception; note localization can only use one (front) camera though

File: nav2_bringup/urdf/single_drum_roller.urdf (robot description, URDF)
Before this commit: robot turtlebot3_waffle, 13 links, 12 joints
Links:
- added link rear_camera_depth_frame
- added link rear_camera_depth_optical_frame
- added link rear_camera_link; collision box size=0.012 0.132 0.020; visual mesh filename=package://turtlebot3_gazebo/models/turtlebot3_common/meshes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
- added link rear_camera_rgb_frame
- added link rear_camera_rgb_optical_frame
- added link rear_camera_scan_frame
Joints:
- added joint rear_camera_depth_joint: type fixed, parent rear_camera_link, child rear_camera_depth_frame, origin xyz=0.005 0.028 0.013 rpy=-1.57 0 -1.57
- added joint rear_camera_depth_optical_joint: type fixed, parent rear_camera_depth_frame, child rear_camera_depth_optical_frame, origin xyz=0 0 0 rpy=0 0 0
- added joint rear_camera_joint: type fixed, parent base_link, child rear_camera_link, origin xyz=-0.064 0 0.094 rpy=0 0 3.14
- added joint rear_camera_rgb_joint: type fixed, parent rear_camera_link, child rear_camera_rgb_frame, origin xyz=0.005 0.018 0.013 rpy=0 0 0
- added joint rear_camera_rgb_optical_joint: type fixed, parent rear_camera_rgb_frame, child rear_camera_rgb_optical_frame, origin xyz=0 0 0 rpy=-1.57 0 -1.57
- added joint rear_camera_scan_joint: type fixed, parent rear_camera_link, child rear_camera_scan_frame, origin xyz=0.005 0.028 0.013 rpy=0 0 0
