Commit message: Initial roller files

File: nav2_bringup/urdf/crewline_roller.urdf (robot description, URDF)
Before this commit: robot crewline_roller, 17 links, 16 joints
Links:
- added link gps_link
- added link roller_link, mass 200.0; collision box size=1.0 2.0 1.0
- link base_link: mass None -> 500.0; geometry collision box size=2.0 2.0 2.0
- link wheel_left_link: mass None -> 10.0; geometry collision cylinder length=0.2 radius=0.2
- link wheel_right_link: mass None -> 10.0; geometry collision cylinder length=0.2 radius=0.2
Joints:
- added joint gps_joint: type fixed, parent base_link, child gps_link, origin xyz=0.0 0 1.0 rpy=0 0 0
- added joint roller_joint: type revolute, parent base_link, child roller_link, origin xyz=1.5 0 -0.5 rpy=0 0 0, axis 0 0 1, limit lower=-0.785 upper=0.785 effort=1000 velocity=1.0
- joint base_joint: origin xyz=0 0 0.010 rpy=0 0 0 -> xyz=0 0 1.0 rpy=0 0 0
- joint front_camera_joint: origin xyz=0.064 0 0.094 rpy=0 0 0 -> xyz=1.0 0 1.0 rpy=0 0 0
- joint imu_joint: origin xyz=0.0 0 0.068 rpy=0 0 0 -> xyz=0.0 0 1.0 rpy=0 0 0
- joint rear_camera_joint: origin xyz=-0.064 0 0.094 rpy=0 0 3.14 -> xyz=-1.0 0 1.0 rpy=0 0 3.14
- joint wheel_left_joint: origin xyz=0.0 0.144 0.023 rpy=-1.57 0 0 -> xyz=0.0 1.0 -0.8 rpy=-1.57 0 0
- joint wheel_right_joint: origin xyz=0.0 -0.144 0.023 rpy=-1.57 0 0 -> xyz=0.0 -1.0 -0.8 rpy=-1.57 0 0

Commit message: Scale down roller to fit into turtlebot map

File: nav2_bringup/urdf/crewline_roller.urdf (robot description, URDF)
Before this commit: robot crewline_roller, 19 links, 18 joints
Links:
- link base_link: mass 500.0 -> 0.5; geometry collision box size=0.2 0.2 0.2
- link roller_link: mass 200.0 -> 0.2; geometry collision box size=0.1 0.2 0.1
- link wheel_left_link: mass 10.0 -> 0.01; geometry collision cylinder length=0.02 radius=0.02
- link wheel_right_link: mass 10.0 -> 0.01; geometry collision cylinder length=0.02 radius=0.02
Joints:
- joint base_joint: origin xyz=0 0 1.0 rpy=0 0 0 -> xyz=0 0 0.1 rpy=0 0 0
- joint front_camera_joint: origin xyz=1.0 0 1.0 rpy=0 0 0 -> xyz=0.1 0 0.1 rpy=0 0 0
- joint gps_joint: origin xyz=0.0 0 1.0 rpy=0 0 0 -> xyz=0.0 0 0.1 rpy=0 0 0
- joint imu_joint: origin xyz=0.0 0 1.0 rpy=0 0 0 -> xyz=0.0 0 0.1 rpy=0 0 0
- joint rear_camera_joint: origin xyz=-1.0 0 1.0 rpy=0 0 3.14 -> xyz=-0.1 0 0.1 rpy=0 0 3.14
- joint roller_joint: origin xyz=1.5 0 -0.5 rpy=0 0 0 -> xyz=0.15 0 -0.05 rpy=0 0 0
- joint wheel_left_joint: origin xyz=0.0 1.0 -0.8 rpy=-1.57 0 0 -> xyz=0.0 0.1 -0.08 rpy=-1.57 0 0
- joint wheel_right_joint: origin xyz=0.0 -1.0 -0.8 rpy=-1.57 0 0 -> xyz=0.0 -0.1 -0.08 rpy=-1.57 0 0

Commit message: Add wheels to roller

File: nav2_bringup/urdf/crewline_roller.urdf (robot description, URDF)
Before this commit: robot crewline_roller, 19 links, 18 joints
Links:
- added link roller_wheel_left_link, mass 0.01; collision cylinder length=0.05 radius=0.05; visual cylinder length=0.05 radius=0.05
- added link roller_wheel_right_link, mass 0.01; collision cylinder length=0.05 radius=0.05; visual cylinder length=0.05 radius=0.05
- link base_link: geometry collision box size=0.2 0.2 0.2; visual box size=0.2 0.2 0.2
- link roller_link: geometry collision box size=0.15 0.2 0.1; visual box size=0.15 0.2 0.1
- link wheel_left_link: geometry collision cylinder length=0.05 radius=0.05; visual cylinder length=0.05 radius=0.05
- link wheel_right_link: geometry collision cylinder length=0.05 radius=0.05; visual cylinder length=0.05 radius=0.05
Joints:
- added joint roller_wheel_left_joint: type continuous, parent roller_link, child roller_wheel_left_link, origin xyz=0.0 0.1 -0.03 rpy=-1.57 0 0, axis 0 0 1
- added joint roller_wheel_right_joint: type continuous, parent roller_link, child roller_wheel_right_link, origin xyz=0.0 -0.1 -0.03 rpy=-1.57 0 0, axis 0 0 1

Commit message: Update joint dimensions

File: nav2_bringup/urdf/crewline_roller.urdf (robot description, URDF)
Before this commit: robot crewline_roller, 21 links, 20 joints
Links:
- link roller_wheel_left_link: geometry collision cylinder length=0.05 radius=0.03; visual cylinder length=0.05 radius=0.03
- link roller_wheel_right_link: geometry collision cylinder length=0.05 radius=0.03; visual cylinder length=0.05 radius=0.03
Joints:
- joint roller_joint: origin xyz=0.15 0 -0.05 rpy=0 0 0 -> xyz=0.175 0 -0.05 rpy=0 0 0

Commit message: Extend base_footprint to roller and use it in nav2 params instead of base_link; reduce vel and accel limits and inflation amounts

File: nav2_bringup/urdf/crewline_roller.urdf (robot description, URDF)
Before this commit: robot crewline_roller, 21 links, 20 joints
Joints:
- joint base_joint: origin xyz=0 0 0.1 rpy=0 0 0 -> xyz=-0.175 0 0.1 rpy=0 0 0
